File: hw/pwr_supply_sheet.sch (KiCad schematic (older format))
At the start: 15 parts

Commit message: making modifications to pcb...
Parts:
- C201, C205: symbol 100nF -> kemet:100nF
- C202: symbol CAP_EEE-FK1H470P -> usevolt:CAP_EEE-FK1H470P
- C203: symbol 10nF -> kemet:10nF
- C204: symbol T491D226K035AT -> kemet:T491D226K035AT
- D201, D203: symbol DIODE_RS07J-GS18 -> usevolt:DIODE_RS07J-GS18
- D202: symbol DIODE_TVS_SMBJ33A-TRDO-214AA -> usevolt:DIODE_TVS_SMBJ33A-TRDO-214AA
- D204, D205: symbol SCHOTTKY_DIODE_V40PW10C -> usevolt:SCHOTTKY_DIODE_V40PW10C
- D206: symbol DIODE_TVS_TPSMD28A -> usevolt:DIODE_TVS_TPSMD28A
- F201: symbol FUSE_MC36211_350MA -> usevolt:FUSE_MC36211_350MA
- L201: symbol IND_744045210 -> usevolt:IND_744045210
- VR201: symbol LM2671SOIC8 -> usevolt:LM2671SOIC8
- VR202: symbol REG_MCP1700 -> usevolt:REG_MCP1700
Changed lines of the file:
@@
-EESchema Schematic File Version 2
-LIBS:csb-rescue
-LIBS:kemet
-LIBS:power
-LIBS:usevolt
-LIBS:wurth_elektronik_LED
-LIBS:yageo
+EESchema Schematic File Version 4
 LIBS:csb-cache
 EELAYER 26 0
@@
 VIN
 $Comp
-L FUSE_MC36211_350MA F201
+L usevolt:FUSE_MC36211_350MA F201
 U 1 1 57B8204F
 P 2500 3850
@@
 $EndComp
 $Comp
-L DIODE_TVS_SMBJ33A-TRDO-214AA D202
+L usevolt:DIODE_TVS_SMBJ33A-TRDO-214AA D202
 U 1 1 57B820C1
 P 2800 4050
@@
 $EndComp
 $Comp
-L 100nF C201
+L kemet:100nF C201
 U 1 1 57B8217A
 P 3400 3950
@@
 $EndComp
 $Comp
-L LM2671SOIC8 VR201
+L usevolt:LM2671SOIC8 VR201
 U 1 1 57B82261
 P 4850 4150
@@
 $EndComp
 $Comp
-L 10nF C203
+L kemet:10nF C203
 U 1 1 57B822C5
 P 5800 3950
@@
 $EndComp
 $Comp
-L DIODE_RS07J-GS18 D203
+L usevolt:DIODE_RS07J-GS18 D203
 U 1 1 57B82329
 P 6200 3950
@@
 $EndComp
 $Comp
-L REG_MCP1700 VR202
+L usevolt:REG_MCP1700 VR202
 U 1 1 57B82857
 P 8000 3950
@@
 $EndComp
 $Comp
-L 100nF C205
+L kemet:100nF C205
 U 1 1 57B82A3F
 P 8600 3950
@@
 $EndComp
 $Comp
-L +5V #PWR205
+L power:+5V #PWR0205
 U 1 1 57B831F8
 P 6850 3600
-F 0 "#PWR205" H 6850 3450 50  0001 C CNN
+F 0 "#PWR0205" H 6850 3450 50  0001 C CNN
 F 1 "+5V" H 6865 3773 50  0000 C CNN
 F 2 "" H 6850 3600 50  0000 C CNN
@@
 $EndComp
 $Comp
-L +3V3 #PWR206
+L power:+3V3 #PWR0206
 U 1 1 57B83259
 P 8600 3600
-F 0 "#PWR206" H 8600 3450 50  0001 C CNN
+F 0 "#PWR0206" H 8600 3450 50  0001 C CNN
 F 1 "+3V3" H 8615 3773 50  0000 C CNN
 F 2 "" H 8600 3600 50  0000 C CNN
@@
 NoConn ~ 4550 4050
 $Comp
-L VDD #PWR203
+L power:VDD #PWR0203
 U 1 1 57B9C56A
 P 3800 2100
-F 0 "#PWR203" H 3800 1950 50  0001 C CNN
+F 0 "#PWR0203" H 3800 1950 50  0001 C CNN
 F 1 "VDD" H 3817 2273 50  0000 C CNN
 F 2 "" H 3800 2100 50  0000 C CNN
@@
 $EndComp
 $Comp
-L PWR_FLAG #FLG201
+L power:PWR_FLAG #FLG0201
 U 1 1 57B9C59C
 P 3800 2300
-F 0 "#FLG201" H 3800 2395 50  0001 C CNN
+F 0 "#FLG0201" H 3800 2395 50  0001 C CNN
 F 1 "PWR_FLAG" H 3800 2523 50  0000 C CNN
 F 2 "" H 3800 2300 50  0000 C CNN
@@
 $EndComp
 $Comp
-L GND #PWR204
+L power:GND #PWR0204
 U 1 1 57B9D351
 P 4300 2350
-F 0 "#PWR204" H 4300 2100 50  0001 C CNN
+F 0 "#PWR0204" H 4300 2100 50  0001 C CNN
 F 1 "GND" H 4305 2177 50  0000 C CNN
 F 2 "" H 4300 2350 50  0000 C CNN
@@
 $EndComp
 $Comp
-L PWR_FLAG #FLG202
+L power:PWR_FLAG #FLG0202
 U 1 1 57B9D3A1
 P 4300 2150
-F 0 "#FLG202" H 4300 2245 50  0001 C CNN
+F 0 "#FLG0202" H 4300 2245 50  0001 C CNN
 F 1 "PWR_FLAG" H 4300 2374 50  0000 C CNN
 F 2 "" H 4300 2150 50  0000 C CNN
@@
 $EndComp
 $Comp
-L GND #PWR201
+L power:GND #PWR0201
 U 1 1 57CF1F5E
 P 2800 4500
-F 0 "#PWR201" H 2800 4250 50  0001 C CNN
+F 0 "#PWR0201" H 2800 4250 50  0001 C CNN
 F 1 "GND" H 2805 4327 50  0000 C CNN
 F 2 "" H 2800 4500 50  0000 C CNN
@@
 $EndComp
 $Comp
-L IND_744045210 L201
+L usevolt:IND_744045210 L201
 U 1 1 58945E39
 P 6500 3850
@@
 $EndComp
 $Comp
-L T491D226K035AT C204
+L kemet:T491D226K035AT C204
 U 1 1 58945F23
 P 6850 4050
@@
 $EndComp
 $Comp
-L DIODE_RS07J-GS18 D201
+L usevolt:DIODE_RS07J-GS18 D201
 U 1 1 5896E2A2
 P 1900 3850
@@
 $EndComp
 $Comp
-L SCHOTTKY_DIODE_V40PW10C D204
+L usevolt:SCHOTTKY_DIODE_V40PW10C D204
 U 1 1 5A0333DC
 P 2050 2900
@@
 $EndComp
 $Comp
-L SCHOTTKY_DIODE_V40PW10C D205
+L usevolt:SCHOTTKY_DIODE_V40PW10C D205
 U 1 1 5A033465
 P 2050 3350
@@
 Connection ~ 1500 3350
 $Comp
-L DIODE_TVS_TPSMD28A D206
+L usevolt:DIODE_TVS_TPSMD28A D206
 U 1 1 5A0E0FEE
 P 3000 3150
@@
 Connection ~ 3000 2850
 $Comp
-L GND #PWR202
+L power:GND #PWR0202
 U 1 1 5A0E10EA
 P 3000 3350
-F 0 "#PWR202" H 3000 3100 50  0001 C CNN
+F 0 "#PWR0202" H 3000 3100 50  0001 C CNN
 F 1 "GND" H 3005 3177 50  0000 C CNN
 F 2 "" H 3000 3350 50  0000 C CNN
@@
 	3000 3350 3000 3250
 $Comp
-L CAP_EEE-FK1H470P C202
+L usevolt:CAP_EEE-FK1H470P C202
 U 1 1 5A0E1265
 P 3800 4050
