File: hw/vn5e010ah.sch (KiCad schematic (older format))
At the start: 4 parts, among them U1001 VN5E010AH

Commit message: Drawing pcb 4.0.0
Parts:
- removed D601: DIODE_RS07J-GS18, usevolt:DO219AB, symbol usevolt:DIODE_RS07J-GS18
- added D4: ZENER_MM3Z3V6T1G, usevolt:SOD-323, symbol usevolt:ZENER_MM3Z3V6T1G
- added R2: 10K, yageo:0603, symbol yageo:10K
Connections:
- net GND: now also D4.2, R2.1 (R1)
- net OUT1: now also R2.2 (R2)
- net SENSE1: now also D4.1
Changed lines of the file:
@@
 AR Path="/5A33548E/59D7E637" Ref="#PWR602"  Part="1"
 AR Path="/5A33648A/59D7E637" Ref="#PWR031"  Part="1"
-F 0 "#PWR0502" H 4600 2850 50  0001 C CNN
+F 0 "#PWR0602" H 4600 2850 50  0001 C CNN
 F 1 "VDD" H 4617 3173 50  0000 C CNN
 F 2 "" H 4600 3000 50  0000 C CNN
@@
 AR Path="/5A33548E/5A014ACD" Ref="#PWR601"  Part="1"
 AR Path="/5A33648A/5A014ACD" Ref="#PWR032"  Part="1"
-F 0 "#PWR0501" H 3850 3350 50  0001 C CNN
+F 0 "#PWR0601" H 3850 3350 50  0001 C CNN
 F 1 "GND" H 3855 3427 50  0000 C CNN
 F 2 "" H 3850 3600 50  0000 C CNN
@@
 AR Path="/5A33548E/5A058D94" Ref="R601"  Part="1"
 AR Path="/5A33648A/5A058D94" Ref="R701"  Part="1"
-F 0 "R501" V 3608 3408 45  0000 L CNN
+F 0 "R601" V 3608 3408 45  0000 L CNN
 F 1 "1K" V 3692 3408 45  0000 L CNN
 F 2 "yageo:0603" H 3630 3500 20  0001 C CNN
@@
 AR Path="/5A019746/5A32CF4A" Ref="U601"  Part="1"
 AR Path="/5A01A445/5A32CF4A" Ref="U701"  Part="1"
-F 0 "U501" H 5250 3747 60  0000 C CNN
+F 0 "U601" H 5250 3747 60  0000 C CNN
 F 1 "VN5E010AH" H 5250 3641 60  0000 C CNN
 F 2 "usevolt:HPAK" H 4950 4250 60  0001 C CNN
@@
 L power:GND #PWR1003
 U 1 1 5A32CF90
-P 4800 3600
+P 4800 3900
 AR Path="/5A1349CF/5A32CF90" Ref="#PWR1003"  Part="1"
 AR Path="/5A14370A/5A32CF90" Ref="#PWR1303"  Part="1"
@@
 AR Path="/5A019746/5A32CF90" Ref="#PWR0603"  Part="1"
 AR Path="/5A01A445/5A32CF90" Ref="#PWR703"  Part="1"
-F 0 "#PWR0503" H 4800 3350 50  0001 C CNN
-F 1 "GND" H 4805 3427 50  0000 C CNN
-F 2 "" H 4800 3600 50  0000 C CNN
-F 3 "" H 4800 3600 50  0000 C CNN
-	1    4800 3600
+F 0 "#PWR0603" H 4800 3650 50  0001 C CNN
+F 1 "GND" H 4805 3727 50  0000 C CNN
+F 2 "" H 4800 3900 50  0000 C CNN
+F 3 "" H 4800 3900 50  0000 C CNN
+	1    4800 3900
 	1    0    0    -1
 $EndComp
@@
 Connection ~ 4800 3500
 Wire Wire Line
-	5700 3200 6200 3200
+	5700 3200 5900 3200
 Wire Wire Line
 	4600 3300 4900 3300
@@
 	3850 3550 3850 3600
 Wire Wire Line
-	4800 3500 4800 3600
+	4800 3500 4800 3800
 $Comp
 L yageo:1K R502
@@
 AR Path="/5A33548E/5B1D30FA" Ref="R?"  Part="1"
 AR Path="/5A33648A/5B1D30FA" Ref="R?"  Part="1"
-F 0 "R502" V 4158 3358 45  0000 L CNN
+F 0 "R602" V 4158 3358 45  0000 L CNN
 F 1 "1K" V 4242 3358 45  0000 L CNN
 F 2 "yageo:0603" H 4180 3450 20  0001 C CNN
@@
 	1    0    0    -1
 $EndComp
-$Comp
-L usevolt:DIODE_RS07J-GS18 D601
-U 1 1 5B1D330E
-P 4300 3850
-AR Path="/5A019746/5B1D330E" Ref="D601"  Part="1"
-AR Path="/5A01611C/5B1D330E" Ref="D501"  Part="1"
-F 0 "D501" H 4250 3710 45  0000 C CNN
-F 1 "DIODE_RS07J-GS18" H 4320 3790 45  0001 L BNN
-F 2 "usevolt:DO219AB" H 4330 4000 20  0001 C CNN
-F 3 "http://www.vishay.com/docs/85742/rs07b.pdf" H 4320 3870 60  0001 C CNN
-F 4 "1864882" H 4920 4470 60  0001 C CNN "2nd Source Part Number"
-F 5 "Digi-Key" H 4620 4170 60  0001 C CNN "1st Source"
-F 6 "Farnell" H 4820 4370 60  0001 C CNN "2nd Source"
-F 7 "RS07J-GS18" H 4520 4070 60  0001 C CNN "Manufacturer Part Number"
-F 8 "RS07J-GS18-ND" H 4720 4270 60  0001 C CNN "1st Source Part Number"
-F 9 "Vishay Semiconductor Diodes Division" H 4420 3970 60  0001 C CNN "Manufacturer"
-	1    4300 3850
-	-1   0    0    1
-$EndComp
-$Comp
-L power:+3V3 #PWR0109
-U 1 1 5B1D3427
-P 4100 3750
-AR Path="/5A019746/5B1D3427" Ref="#PWR0109"  Part="1"
-AR Path="/5A01611C/5B1D3427" Ref="#PWR0108"  Part="1"
-F 0 "#PWR0108" H 4100 3600 50  0001 C CNN
-F 1 "+3V3" H 4115 3923 50  0000 C CNN
-F 2 "" H 4100 3750 50  0000 C CNN
-F 3 "" H 4100 3750 50  0000 C CNN
-	1    4100 3750
-	1    0    0    -1
-$EndComp
-Wire Wire Line
-	4100 3750 4100 3850
-Wire Wire Line
-	4100 3850 4200 3850
-Wire Wire Line
-	4500 3850 4600 3850
-Wire Wire Line
-	4600 3850 4600 3450
+Wire Wire Line
+	4600 3550 4600 3450
 Connection ~ 4600 3450
+$Comp
+L usevolt:ZENER_MM3Z3V6T1G D4
+U 1 1 5BABCC09
+P 4600 3600
+AR Path="/5A019746/5BABCC09" Ref="D4"  Part="1"
+AR Path="/5A01611C/5BABCC09" Ref="D3"  Part="1"
+F 0 "D4" V 4525 3522 45  0000 R CNN
+F 1 "ZENER_MM3Z3V6T1G" H 4875 3975 45  0001 L BNN
+F 2 "usevolt:SOD-323" H 4575 3975 20  0001 C CNN
+F 3 "http://www.mouser.com/ds/2/308/MM3Z2V4T1-D-269162.pdf" H 4950 4175 60  0001 C CNN
+F 4 "Mouser" H 4920 3920 60  0001 C CNN "1st Source"
+F 5 "MM3Z3V6T1G" H 4820 3820 60  0001 C CNN "Manufacturer Part Number"
+F 6 "863-MM3Z3V6T1G" H 5020 4020 60  0001 C CNN "1st Source Part Number"
+F 7 "ON Semiconductor" H 4875 4075 60  0001 C CNN "Manufacturer"
+	1    4600 3600
+	0    -1   -1   0
+$EndComp
+Wire Wire Line
+	4600 3800 4800 3800
+Connection ~ 4800 3800
+Wire Wire Line
+	4800 3800 4800 3900
+$Comp
+L yageo:10K R2
+U 1 1 5BABD3C0
+P 5900 3400
+AR Path="/5A019746/5BABD3C0" Ref="R2"  Part="1"
+AR Path="/5A01611C/5BABD3C0" Ref="R1"  Part="1"
+F 0 "R2" V 5908 3458 45  0000 L CNN
+F 1 "10K" V 5992 3458 45  0000 L CNN
+F 2 "yageo:0603" H 5930 3550 20  0001 C CNN
+F 3 "" H 5869 3439 60  0001 C CNN
+F 4 "" H 6269 3839 60  0001 C CNN "1st Source Part Number"
+F 5 "Digikey" H 6169 3739 60  0001 C CNN "1st Source"
+F 6 "RC0603FR-0710KL" H 6069 3639 60  0001 C CNN "Manufacturer Part Number"
+F 7 "YAGEO" H 5969 3539 60  0001 C CNN "Manufacturer"
+	1    5900 3400
+	0    1    1    0
+$EndComp
+Wire Wire Line
+	5900 3300 5900 3200
+Connection ~ 5900 3200
+Wire Wire Line
+	5900 3200 6200 3200
+$Comp
+L power:GND #PWR0108
+U 1 1 5BABD6AD
+P 5900 3700
+AR Path="/5A019746/5BABD6AD" Ref="#PWR0108"  Part="1"
+AR Path="/5A01611C/5BABD6AD" Ref="#PWR0107"  Part="1"
+F 0 "#PWR0108" H 5900 3450 50  0001 C CNN
+F 1 "GND" H 5905 3527 50  0000 C CNN
+F 2 "" H 5900 3700 50  0000 C CNN
+F 3 "" H 5900 3700 50  0000 C CNN
+	1    5900 3700
+	1    0    0    -1
+$EndComp
+Wire Wire Line
+	5900 3700 5900 3600
 $EndSCHEMATC
