File: hw/lpc1549.sch (KiCad schematic (older format))
At the start: 17 parts, among them J301 ARM_JTAG_SWD_HEADER_10_PINSMD, U301 LPC1549JBD64, U302 MCP2551_SOIC8, X301 XTAL_7A-12.000MAAJ-T

Commit message: making modifications to pcb...
Parts:
- C301, C302, C303, C304, C305, C306, C309: symbol 100nF -> kemet:100nF
- C307, C308: symbol 18pF -> kemet:18pF
- J301: symbol ARM_JTAG_SWD_HEADER_10_PINSMD -> usevolt:ARM_JTAG_SWD_HEADER_10_PINSMD
- R301, R302, R303, R304: symbol 10K -> yageo:10K
- U301: symbol LPC1549JBD64 -> usevolt:LPC1549JBD64
- U302: symbol MCP2551_SOIC8 -> usevolt:MCP2551_SOIC8
- X301: symbol XTAL_7A-12.000MAAJ-T -> usevolt:XTAL_7A-12.000MAAJ-T
Connections:
- net +5V: now also U302.3 (VDD); no longer U302.P$3 (VDD)
- net CANH: now also U302.7 (CANH); no longer U302.P$7 (CANH)
- net CANL: now also U302.6 (CANL); no longer U302.P$6 (CANL)
- net CAN_RX: now also U302.4 (RXD); no longer U302.P$4 (RXD)
- net CAN_TX: now also U302.1 (TXD); no longer U302.P$1 (TXD)
- net GND: now also U301.P$41 (VBAT), U302.2 (VSS), U302.8 (RS/GND); no longer U301.P$39 (PIO0_17/WAKEUP/!TRST), U302.P$2 (VSS), U302.P$8 (RS/GND)
- net at J301.P$2 (TMS/SWDIO), R303.1 (R1): now also U301.P$44 (SWDIO/PIO0_20/SCT1_OUT6/TMS)
- net at J301.P$4 (TCK/SWDCLK), R304.1 (R1): now also U301.P$40 (SWCLK/PIO0_19/TCK)
Changed lines of the file:
@@
-EESchema Schematic File Version 2
-LIBS:csb-rescue
-LIBS:kemet
-LIBS:power
-LIBS:usevolt
-LIBS:wurth_elektronik_LED
-LIBS:yageo
+EESchema Schematic File Version 4
 LIBS:csb-cache
 EELAYER 26 0
@@
 $EndDescr
 $Comp
-L 100nF C306
+L kemet:100nF C306
 U 1 1 57E685B4
 P 4400 4100
@@
 $EndComp
 $Comp
-L 100nF C305
+L kemet:100nF C305
 U 1 1 57E68621
 P 4050 4100
@@
 $EndComp
 $Comp
-L 100nF C304
+L kemet:100nF C304
 U 1 1 57E68672
 P 3700 4100
@@
 $EndComp
 $Comp
-L 100nF C303
+L kemet:100nF C303
 U 1 1 57E686C7
 P 3350 4100
@@
 $EndComp
 $Comp
-L 100nF C302
+L kemet:100nF C302
 U 1 1 57E6871C
 P 3000 4100
@@
 $EndComp
 $Comp
-L +3V3 #PWR301
+L power:+3V3 #PWR0301
 U 1 1 57E689A3
 P 3000 3850
-F 0 "#PWR301" H 3000 3700 50  0001 C CNN
+F 0 "#PWR0301" H 3000 3700 50  0001 C CNN
 F 1 "+3V3" H 3015 4023 50  0000 C CNN
 F 2 "" H 3000 3850 50  0000 C CNN
@@
 $EndComp
 $Comp
-L GND #PWR302
+L power:GND #PWR0302
 U 1 1 57E689C9
 P 3000 4450
-F 0 "#PWR302" H 3000 4200 50  0001 C CNN
+F 0 "#PWR0302" H 3000 4200 50  0001 C CNN
 F 1 "GND" H 3005 4277 50  0000 C CNN
 F 2 "" H 3000 4450 50  0000 C CNN
@@
 $EndComp
 $Comp
-L XTAL_7A-12.000MAAJ-T X301
+L usevolt:XTAL_7A-12.000MAAJ-T X301
 U 1 1 57E6956F
 P 6650 2850
@@
 $EndComp
 $Comp
-L 18pF C307
+L kemet:18pF C307
 U 1 1 57E695FA
 P 6950 2650
@@
 $EndComp
 $Comp
-L 18pF C308
+L kemet:18pF C308
 U 1 1 57E69648
 P 6950 2950
@@
 $EndComp
 $Comp
-L GND #PWR304
+L power:GND #PWR0304
 U 1 1 57E697A1
 P 7400 3000
-F 0 "#PWR304" H 7400 2750 50  0001 C CNN
+F 0 "#PWR0304" H 7400 2750 50  0001 C CNN
 F 1 "GND" H 7405 2827 50  0000 C CNN
 F 2 "" H 7400 3000 50  0000 C CNN
@@
 $EndComp
 $Comp
-L GND #PWR303
+L power:GND #PWR0303
 U 1 1 57E69A8B
 P 6700 3250
-F 0 "#PWR303" H 6700 3000 50  0001 C CNN
+F 0 "#PWR0303" H 6700 3000 50  0001 C CNN
 F 1 "GND" H 6705 3077 50  0000 C CNN
 F 2 "" H 6700 3250 50  0000 C CNN
@@
 $EndComp
 $Comp
-L GND #PWR305
+L power:GND #PWR0305
 U 1 1 5891FBFB
 P 8600 4400
-F 0 "#PWR305" H 8600 4150 50  0001 C CNN
+F 0 "#PWR0305" H 8600 4150 50  0001 C CNN
 F 1 "GND" H 8605 4227 50  0000 C CNN
 F 2 "" H 8600 4400 50  0000 C CNN
@@
 $EndComp
 $Comp
-L +3V3 #PWR306
+L power:+3V3 #PWR0306
 U 1 1 5891FCDE
 P 8650 3350
-F 0 "#PWR306" H 8650 3200 50  0001 C CNN
+F 0 "#PWR0306" H 8650 3200 50  0001 C CNN
 F 1 "+3V3" H 8665 3523 50  0000 C CNN
 F 2 "" H 8650 3350 50  0000 C CNN
@@
 RESET
 $Comp
-L 10K R303
+L yageo:10K R303
 U 1 1 589226EB
 P 8150 3450
@@
 $EndComp
 $Comp
-L 10K R304
+L yageo:10K R304
 U 1 1 58922760
 P 8400 3500
@@
 Connection ~ 8650 3350
 $Comp
-L GND #PWR308
+L power:GND #PWR0308
 U 1 1 58C01588
 P 10100 6150
-F 0 "#PWR308" H 10100 5900 50  0001 C CNN
+F 0 "#PWR0308" H 10100 5900 50  0001 C CNN
 F 1 "GND" H 10105 5977 50  0000 C CNN
 F 2 "" H 10100 6150 50  0000 C CNN
@@
 $EndComp
 $Comp
-L 100nF C?
+L kemet:100nF C?
 U 1 1 58C01592
 P 10200 5800
@@
 	9550 5250 8650 5250
 $Comp
-L 100nF C301
+L kemet:100nF C301
 U 1 1 58D0A5A6
 P 2650 4100
@@
 Connection ~ 4400 4300
 $Comp
-L ARM_JTAG_SWD_HEADER_10_PINSMD J301
+L usevolt:ARM_JTAG_SWD_HEADER_10_PINSMD J301
 U 1 1 5953ECE3
 P 8850 3850
@@
 Connection ~ 9750 6000
 $Comp
-L 10K R301
+L yageo:10K R301
 U 1 1 5957A035
 P 6600 2450
@@
 WIPER_POS
 $Comp
-L 10K R302
+L yageo:10K R302
 U 1 1 5957B1E8
 P 6850 2550
@@
 	9600 5700 10200 5700
 $Comp
-L +5V #PWR307
+L power:+5V #PWR0307
 U 1 1 595E0BE4
 P 10100 5600
-F 0 "#PWR307" H 10100 5450 50  0001 C CNN
+F 0 "#PWR0307" H 10100 5450 50  0001 C CNN
 F 1 "+5V" H 10115 5773 50  0000 C CNN
 F 2 "" H 10100 5600 50  0000 C CNN
@@
 Connection ~ 10100 5700
 $Comp
-L LPC1549JBD64 U301
+L usevolt:LPC1549JBD64 U301
 U 1 1 5A00BF20
 P 5100 2650
@@
 	8050 3550 8050 3850
 $Comp
-L MCP2551_SOIC8 U302
+L usevolt:MCP2551_SOIC8 U302
 U 1 1 5A031B21
 P 9300 5800

Commit message: pcb 3.4.0 created, ready for order
Connections:
- net at R301.2 (R2): now also U301.P$15 (PIO1_1/ADC1_0); no longer U301.P$33 (PIO1_4/ADC1_10)
- net at R302.2 (R2): now also U301.P$16 (PIO0_9/ADC1_1/TDI); no longer U301.P$34 (PIO1_5/ADC1_11)
Other:
- moved on the sheet: R301, R302
Changed lines of the file:
@@
 $EndComp
 Wire Wire Line
-	4400 4300 4400 4800
-Wire Wire Line
-	4400 4400 4600 4400
+	4400 4300 4400 4400
+Wire Wire Line
+	4400 4400 4500 4400
 Wire Wire Line
 	4600 4300 4500 4300
@@
 Connection ~ 4500 4400
 Wire Wire Line
-	2650 4000 4600 4000
+	2650 4000 3000 4000
 Connection ~ 4400 4000
 Connection ~ 4050 4000
@@
 Connection ~ 3350 4000
 Wire Wire Line
-	2650 4300 4400 4300
+	2650 4300 3000 4300
 Connection ~ 3350 4300
 Connection ~ 3700 4300
@@
 Connection ~ 4400 3450
 Wire Wire Line
-	4400 3350 4400 4000
-Wire Wire Line
-	6500 2950 6850 2950
+	4400 3350 4400 3450
+Wire Wire Line
+	6500 2950 6650 2950
 Wire Wire Line
 	6500 2950 6500 2850
@@
 	6500 2750 6500 2650
 Wire Wire Line
-	6500 2650 6850 2650
+	6500 2650 6650 2650
 Connection ~ 6650 2650
 Wire Wire Line
 	7150 2650 7400 2650
 Wire Wire Line
-	7400 2650 7400 3000
+	7400 2650 7400 2950
 Wire Wire Line
 	7400 2950 7150 2950
@@
 	7000 5050 6400 5050
 Wire Wire Line
-	8050 3850 8750 3850
-Wire Wire Line
-	6400 3650 8750 3650
-Wire Wire Line
-	8600 3750 8600 4400
+	8050 3850 8400 3850
+Wire Wire Line
+	6400 3650 8150 3650
+Wire Wire Line
+	8600 3750 8600 3950
 Wire Wire Line
 	8600 3950 8750 3950
@@
 Connection ~ 8400 3850
 Wire Wire Line
-	8150 3350 8650 3350
+	8150 3350 8400 3350
 Wire Wire Line
 	8400 3400 8400 3350
@@
 $EndComp
 Wire Wire Line
-	9600 6000 10200 6000
+	9600 6000 9750 6000
 Wire Wire Line
 	10100 6000 10100 6150
@@
 L yageo:10K R301
 U 1 1 5957A035
-P 6600 2450
-F 0 "R301" H 6650 2634 45  0000 C CNN
-F 1 "10K" H 6650 2550 45  0000 C CNN
-F 2 "multicomp:0603" H 6630 2600 20  0001 C CNN
-F 3 "http://www.farnell.com/datasheets/1788326.pdf?_ga=1.214208087.1948984246.1460023966" H 6569 2489 60  0001 C CNN
-F 4 "9330399" H 6969 2889 60  0001 C CNN "1st Source Part Number"
-F 5 "Farnell" H 6869 2789 60  0001 C CNN "1st Source"
-F 6 "MC0063W0603110K" H 6769 2689 60  0001 C CNN "Manufacturer Part Number"
-F 7 "MULTICOMP" H 6669 2589 60  0001 C CNN "Manufacturer"
-	1    6600 2450
-	1    0    0    1
-$EndComp
-Wire Wire Line
-	6500 2450 6400 2450
-Wire Wire Line
-	6800 2450 7350 2450
-Text HLabel 7350 2450 2    60   Input ~ 0
+P 4400 4950
+F 0 "R301" H 4450 5134 45  0000 C CNN
+F 1 "10K" H 4450 5050 45  0000 C CNN
+F 2 "multicomp:0603" H 4430 5100 20  0001 C CNN
+F 3 "http://www.farnell.com/datasheets/1788326.pdf?_ga=1.214208087.1948984246.1460023966" H 4369 4989 60  0001 C CNN
+F 4 "9330399" H 4769 5389 60  0001 C CNN "1st Source Part Number"
+F 5 "Farnell" H 4669 5289 60  0001 C CNN "1st Source"
+F 6 "MC0063W0603110K" H 4569 5189 60  0001 C CNN "Manufacturer Part Number"
+F 7 "MULTICOMP" H 4469 5089 60  0001 C CNN "Manufacturer"
+	1    4400 4950
+	-1   0    0    1
+$EndComp
+Wire Wire Line
+	4500 4950 4600 4950
+Wire Wire Line
+	4200 4950 3650 4950
+Text HLabel 3650 4950 0    60   Input ~ 0
 WIPER_POS
 $Comp
 L yageo:10K R302
 U 1 1 5957B1E8
-P 6850 2550
-F 0 "R302" H 6900 2734 45  0000 C CNN
-F 1 "10K" H 6900 2650 45  0000 C CNN
-F 2 "multicomp:0603" H 6880 2700 20  0001 C CNN
-F 3 "http://www.farnell.com/datasheets/1788326.pdf?_ga=1.214208087.1948984246.1460023966" H 6819 2589 60  0001 C CNN
-F 4 "9330399" H 7219 2989 60  0001 C CNN "1st Source Part Number"
-F 5 "Farnell" H 7119 2889 60  0001 C CNN "1st Source"
-F 6 "MC0063W0603110K" H 7019 2789 60  0001 C CNN "Manufacturer Part Number"
-F 7 "MULTICOMP" H 6919 2689 60  0001 C CNN "Manufacturer"
-	1    6850 2550
-	1    0    0    1
-$EndComp
-Wire Wire Line
-	6750 2550 6400 2550
-Wire Wire Line
-	7050 2550 7350 2550
-Text HLabel 7350 2550 2    60   Input ~ 0
+P 4150 5050
+F 0 "R302" H 4200 5234 45  0000 C CNN
+F 1 "10K" H 4200 5150 45  0000 C CNN
+F 2 "multicomp:0603" H 4180 5200 20  0001 C CNN
+F 3 "http://www.farnell.com/datasheets/1788326.pdf?_ga=1.214208087.1948984246.1460023966" H 4119 5089 60  0001 C CNN
+F 4 "9330399" H 4519 5489 60  0001 C CNN "1st Source Part Number"
+F 5 "Farnell" H 4419 5389 60  0001 C CNN "1st Source"
+F 6 "MC0063W0603110K" H 4319 5289 60  0001 C CNN "Manufacturer Part Number"
+F 7 "MULTICOMP" H 4219 5189 60  0001 C CNN "Manufacturer"
+	1    4150 5050
+	-1   0    0    1
+$EndComp
+Wire Wire Line
+	4250 5050 4600 5050
+Wire Wire Line
+	3950 5050 3650 5050
+Text HLabel 3650 5050 0    60   Input ~ 0
 COOLER_P
 Wire Wire Line
@@
 COOLER_SENSE
 Wire Wire Line
-	9600 5700 10200 5700
+	9600 5700 10100 5700
 $Comp
 L power:+5V #PWR0307
@@
 	-1   0    0    -1
 $EndComp
+Wire Wire Line
+	4500 4400 4600 4400
+Wire Wire Line
+	4400 4000 4600 4000
+Wire Wire Line
+	4050 4000 4400 4000
+Wire Wire Line
+	3700 4000 4050 4000
+Wire Wire Line
+	3350 4000 3700 4000
+Wire Wire Line
+	3350 4300 3700 4300
+Wire Wire Line
+	3700 4300 4050 4300
+Wire Wire Line
+	4050 4300 4400 4300
+Wire Wire Line
+	4400 4400 4400 4500
+Wire Wire Line
+	4400 4500 4400 4600
+Wire Wire Line
+	4400 4600 4400 4700
+Wire Wire Line
+	4400 4700 4400 4800
+Wire Wire Line
+	4400 3900 4400 4000
+Wire Wire Line
+	4400 3800 4400 3900
+Wire Wire Line
+	4400 3700 4400 3800
+Wire Wire Line
+	4400 3600 4400 3700
+Wire Wire Line
+	4400 3450 4400 3600
+Wire Wire Line
+	6650 2950 6850 2950
+Wire Wire Line
+	6650 2650 6850 2650
+Wire Wire Line
+	7400 2950 7400 3000
+Wire Wire Line
+	8600 3950 8600 4400
+Wire Wire Line
+	8150 3650 8750 3650
+Wire Wire Line
+	8400 3850 8750 3850
+Wire Wire Line
+	8400 3350 8650 3350
+Wire Wire Line
+	10100 6000 10200 6000
+Wire Wire Line
+	3000 4300 3350 4300
+Wire Wire Line
+	3000 4000 3350 4000
+Wire Wire Line
+	9750 6000 10100 6000
+Wire Wire Line
+	10100 5700 10200 5700
 $EndSCHEMATC
