File: hw/csb.sch (KiCad schematic (older format))
At the start: 2 parts, among them J101 AMPSEAL_23_POS_VERT_BLUE_SEAL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, J102 AMPSEAL_8_POS_VERT_BLACK_SEAL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

Commit message: making modifications to pcb...
Parts:
- J101: symbol AMPSEAL_23_POS_VERT_BLUE_SEALED_1-776228-5-RESCUE-csb -> csb-rescue:AMPSEAL_23_POS_VERT_BLUE_SEALED_1-776228-5-RESCUE-csb
- J102: symbol AMPSEAL_8_POS_VERT_BLACK_SEALED_1-776276-1-RESCUE-csb -> csb-rescue:AMPSEAL_8_POS_VERT_BLACK_SEALED_1-776276-1-RESCUE-csb
Changed lines of the file:
@@
-EESchema Schematic File Version 2
-LIBS:csb-rescue
-LIBS:kemet
-LIBS:power
-LIBS:usevolt
-LIBS:wurth_elektronik_LED
-LIBS:yageo
+EESchema Schematic File Version 4
 LIBS:csb-cache
 EELAYER 26 0
@@
 $EndSheet
 $Comp
-L VDD #PWR101
+L power:VDD #PWR0101
 U 1 1 59541057
 P 3450 1150
-F 0 "#PWR101" H 3450 1000 50  0001 C CNN
+F 0 "#PWR0101" H 3450 1000 50  0001 C CNN
 F 1 "VDD" H 3467 1323 50  0000 C CNN
 F 2 "" H 3450 1150 50  0000 C CNN
@@
 $EndComp
 $Comp
-L +5V #PWR102
+L power:+5V #PWR0102
 U 1 1 595410AC
 P 3650 1150
-F 0 "#PWR102" H 3650 1000 50  0001 C CNN
+F 0 "#PWR0102" H 3650 1000 50  0001 C CNN
 F 1 "+5V" H 3665 1323 50  0000 C CNN
 F 2 "" H 3650 1150 50  0000 C CNN
@@
 $EndComp
 $Comp
-L +3V3 #PWR103
+L power:+3V3 #PWR0103
 U 1 1 595410EA
 P 3850 1150
-F 0 "#PWR103" H 3850 1000 50  0001 C CNN
+F 0 "#PWR0103" H 3850 1000 50  0001 C CNN
 F 1 "+3V3" H 3865 1323 50  0000 C CNN
 F 2 "" H 3850 1150 50  0000 C CNN
@@
 $EndComp
 $Comp
-L AMPSEAL_8_POS_VERT_BLACK_SEALED_1-776276-1-RESCUE-csb J102
+L csb-rescue:AMPSEAL_8_POS_VERT_BLACK_SEALED_1-776276-1-RESCUE-csb J102
 U 1 1 59541432
 P 900 1550
@@
 $EndComp
 $Comp
-L AMPSEAL_8_POS_VERT_BLACK_SEALED_1-776276-1-RESCUE-csb J102
+L csb-rescue:AMPSEAL_8_POS_VERT_BLACK_SEALED_1-776276-1-RESCUE-csb J102
 U 2 1 595414CB
 P 900 1700
@@
 $EndComp
 $Comp
-L AMPSEAL_8_POS_VERT_BLACK_SEALED_1-776276-1-RESCUE-csb J102
+L csb-rescue:AMPSEAL_8_POS_VERT_BLACK_SEALED_1-776276-1-RESCUE-csb J102
 U 3 1 5954155F
 P 900 1850
@@
 $EndComp
 $Comp
-L AMPSEAL_8_POS_VERT_BLACK_SEALED_1-776276-1-RESCUE-csb J102
+L csb-rescue:AMPSEAL_8_POS_VERT_BLACK_SEALED_1-776276-1-RESCUE-csb J102
 U 4 1 595415DF
 P 900 2000
@@
 $EndComp
 $Comp
-L AMPSEAL_8_POS_VERT_BLACK_SEALED_1-776276-1-RESCUE-csb J102
+L csb-rescue:AMPSEAL_8_POS_VERT_BLACK_SEALED_1-776276-1-RESCUE-csb J102
 U 5 1 59541657
 P 900 2150
@@
 $EndComp
 $Comp
-L AMPSEAL_8_POS_VERT_BLACK_SEALED_1-776276-1-RESCUE-csb J102
+L csb-rescue:AMPSEAL_8_POS_VERT_BLACK_SEALED_1-776276-1-RESCUE-csb J102
 U 6 1 595416D1
 P 900 2300
@@
 $EndComp
 $Comp
-L AMPSEAL_8_POS_VERT_BLACK_SEALED_1-776276-1-RESCUE-csb J102
+L csb-rescue:AMPSEAL_8_POS_VERT_BLACK_SEALED_1-776276-1-RESCUE-csb J102
 U 7 1 5954174D
 P 900 2450
@@
 $EndComp
 $Comp
-L AMPSEAL_8_POS_VERT_BLACK_SEALED_1-776276-1-RESCUE-csb J102
+L csb-rescue:AMPSEAL_8_POS_VERT_BLACK_SEALED_1-776276-1-RESCUE-csb J102
 U 8 1 595417CB
 P 900 2600
@@
 COOLER_30A
 $Comp
-L AMPSEAL_23_POS_VERT_BLUE_SEALED_1-776228-5-RESCUE-csb J101
+L csb-rescue:AMPSEAL_23_POS_VERT_BLUE_SEALED_1-776228-5-RESCUE-csb J101
 U 1 1 595D3228
 P 10900 2300
@@
 $EndComp
 $Comp
-L AMPSEAL_23_POS_VERT_BLUE_SEALED_1-776228-5-RESCUE-csb J101
+L csb-rescue:AMPSEAL_23_POS_VERT_BLUE_SEALED_1-776228-5-RESCUE-csb J101
 U 2 1 595D3550
 P 11100 2400
@@
 $EndComp
 $Comp
-L AMPSEAL_23_POS_VERT_BLUE_SEALED_1-776228-5-RESCUE-csb J101
+L csb-rescue:AMPSEAL_23_POS_VERT_BLUE_SEALED_1-776228-5-RESCUE-csb J101
 U 3 1 595D36E2
 P 11100 2900
@@
 $EndComp
 $Comp
-L AMPSEAL_23_POS_VERT_BLUE_SEALED_1-776228-5-RESCUE-csb J101
+L csb-rescue:AMPSEAL_23_POS_VERT_BLUE_SEALED_1-776228-5-RESCUE-csb J101
 U 4 1 595D386E
 P 750 4400
@@
 $EndComp
 $Comp
-L AMPSEAL_23_POS_VERT_BLUE_SEALED_1-776228-5-RESCUE-csb J101
+L csb-rescue:AMPSEAL_23_POS_VERT_BLUE_SEALED_1-776228-5-RESCUE-csb J101
 U 5 1 595D39FC
 P 750 4550
@@
 $EndComp
 $Comp
-L AMPSEAL_23_POS_VERT_BLUE_SEALED_1-776228-5-RESCUE-csb J101
+L csb-rescue:AMPSEAL_23_POS_VERT_BLUE_SEALED_1-776228-5-RESCUE-csb J101
 U 6 1 595D3B8C
 P 750 4700
@@
 $EndComp
 $Comp
-L AMPSEAL_23_POS_VERT_BLUE_SEALED_1-776228-5-RESCUE-csb J101
+L csb-rescue:AMPSEAL_23_POS_VERT_BLUE_SEALED_1-776228-5-RESCUE-csb J101
 U 7 1 595D3D22
 P 750 4850
@@
 $EndComp
 $Comp
-L AMPSEAL_23_POS_VERT_BLUE_SEALED_1-776228-5-RESCUE-csb J101
+L csb-rescue:AMPSEAL_23_POS_VERT_BLUE_SEALED_1-776228-5-RESCUE-csb J101
 U 9 1 595D404C
 P 10900 2100
@@
 $EndComp
 $Comp
-L AMPSEAL_23_POS_VERT_BLUE_SEALED_1-776228-5-RESCUE-csb J101
+L csb-rescue:AMPSEAL_23_POS_VERT_BLUE_SEALED_1-776228-5-RESCUE-csb J101
 U 10 1 595D41E8
 P 10900 2800
@@
 $EndComp
 $Comp
-L AMPSEAL_23_POS_VERT_BLUE_SEALED_1-776228-5-RESCUE-csb J101
+L csb-rescue:AMPSEAL_23_POS_VERT_BLUE_SEALED_1-776228-5-RESCUE-csb J101
 U 11 1 595D4382
 P 10900 3000
@@
 $EndComp
 $Comp
-L AMPSEAL_23_POS_VERT_BLUE_SEALED_1-776228-5-RESCUE-csb J101
+L csb-rescue:AMPSEAL_23_POS_VERT_BLUE_SEALED_1-776228-5-RESCUE-csb J101
 U 12 1 595D451E
 P 750 5500
@@
 $EndComp
 $Comp
-L AMPSEAL_23_POS_VERT_BLUE_SEALED_1-776228-5-RESCUE-csb J101
+L csb-rescue:AMPSEAL_23_POS_VERT_BLUE_SEALED_1-776228-5-RESCUE-csb J101
 U 13 1 595D46C0
 P 3650 3850
@@
 $EndComp
 $Comp
-L AMPSEAL_23_POS_VERT_BLUE_SEALED_1-776228-5-RESCUE-csb J101
+L csb-rescue:AMPSEAL_23_POS_VERT_BLUE_SEALED_1-776228-5-RESCUE-csb J101
 U 14 1 595D4862
 P 750 5750
@@
 $EndComp
 $Comp
-L AMPSEAL_23_POS_VERT_BLUE_SEALED_1-776228-5-RESCUE-csb J101
+L csb-rescue:AMPSEAL_23_POS_VERT_BLUE_SEALED_1-776228-5-RESCUE-csb J101
 U 15 1 595D4A2A
 P 3450 3950
@@
 $EndComp
 $Comp
-L AMPSEAL_23_POS_VERT_BLUE_SEALED_1-776228-5-RESCUE-csb J101
+L csb-rescue:AMPSEAL_23_POS_VERT_BLUE_SEALED_1-776228-5-RESCUE-csb J101
 U 16 1 595D4BCE
 P 11100 2200
@@
 $EndComp
 $Comp
-L AMPSEAL_23_POS_VERT_BLUE_SEALED_1-776228-5-RESCUE-csb J101
+L csb-rescue:AMPSEAL_23_POS_VERT_BLUE_SEALED_1-776228-5-RESCUE-csb J101
 U 17 1 595D4D74
 P 11100 2700
@@
 $EndComp
 $Comp
-L AMPSEAL_23_POS_VERT_BLUE_SEALED_1-776228-5-RESCUE-csb J101
+L csb-rescue:AMPSEAL_23_POS_VERT_BLUE_SEALED_1-776228-5-RESCUE-csb J101
 U 18 1 595D4F1C
 P 11100 3400
@@
 $EndComp
 $Comp
-L AMPSEAL_23_POS_VERT_BLUE_SEALED_1-776228-5-RESCUE-csb J101
+L csb-rescue:AMPSEAL_23_POS_VERT_BLUE_SEALED_1-776228-5-RESCUE-csb J101
 U 19 1 595D50C6
 P 10850 3200
@@
 $EndComp
 $Comp
-L AMPSEAL_23_POS_VERT_BLUE_SEALED_1-776228-5-RESCUE-csb J101
+L csb-rescue:AMPSEAL_23_POS_VERT_BLUE_SEALED_1-776228-5-RESCUE-csb J101
 U 20 1 595D5274
 P 11100 4100
@@
 $EndComp
 $Comp
-L AMPSEAL_23_POS_VERT_BLUE_SEALED_1-776228-5-RESCUE-csb J101
+L csb-rescue:AMPSEAL_23_POS_VERT_BLUE_SEALED_1-776228-5-RESCUE-csb J101
 U 21 1 595D5426
 P 10900 3900
@@
 $EndComp
 $Comp
-L AMPSEAL_23_POS_VERT_BLUE_SEALED_1-776228-5-RESCUE-csb J101
+L csb-rescue:AMPSEAL_23_POS_VERT_BLUE_SEALED_1-776228-5-RESCUE-csb J101
 U 22 1 595D55F0
 P 10900 4600
@@
 $EndComp
 $Comp
-L AMPSEAL_23_POS_VERT_BLUE_SEALED_1-776228-5-RESCUE-csb J101
+L csb-rescue:AMPSEAL_23_POS_VERT_BLUE_SEALED_1-776228-5-RESCUE-csb J101
 U 23 1 595D57A2
 P 11100 4700
@@
 U 5A01A445
 F0 "Sheet5A01A444" 60
-F1 "vn5e010ah.sch" 60
+F1 "vn5e010ah_double.sch" 60
 F2 "OUT1" O R 9900 4600 60
 F3 "IN1" I L 9050 4600 60
@@
 	1000 1550 1600 1550
 Wire Wire Line
-	1600 1300 1600 2300
+	1600 1300 1600 1550
 Wire Wire Line
 	1600 1300 2050 1300
@@
 Connection ~ 1600 1550
 Wire Wire Line
-	9900 2200 11000 2200
+	9900 2200 10750 2200
 Wire Wire Line
 	9900 3400 11000 3400
 Wire Wire Line
-	9900 2700 11000 2700
+	9900 2700 10750 2700
 Wire Wire Line
 	9900 4100 11000 4100
@@
 	9900 3900 10800 3900
 Wire Wire Line
-	9900 4600 10800 4600
+	9900 4600 10650 4600
 Wire Wire Line
 	11000 4700 10650 4700
@@
 	10800 2100 10750 2100
 Wire Wire Line
-	10750 2100 10750 2400
+	10750 2100 10750 2200
 Connection ~ 10750 2200
 Wire Wire Line
@@
 Connection ~ 10750 2300
 Wire Wire Line
-	10750 2700 10750 3000
+	10750 2700 10750 2800
 Wire Wire Line
 	10750 3000 10800 3000
@@
 Wire Wire Line
 	6400 3100 8650 3100
+Wire Wire Line
+	1600 1550 1600 1850
+Wire Wire Line
+	10650 4600 10800 4600
+Wire Wire Line
+	1600 1850 1600 2300
+Wire Wire Line
+	10750 2200 11000 2200
+Wire Wire Line
+	10750 2200 10750 2300
+Wire Wire Line
+	10750 2300 10750 2400
+Wire Wire Line
+	10750 2700 11000 2700
+Wire Wire Line
+	10750 2900 10750 3000
+Wire Wire Line
+	10750 2800 10750 2900
 $EndSCHEMATC

Commit message: pcb 3.6.0 created, with double fets in work & drive lights
Changed lines of the file:
@@
 U 5A01611C
 F0 "Sheet5A01611B" 60
-F1 "vn5e010ah.sch" 60
+F1 "vn5e010ah_double.sch" 60
 F2 "OUT1" O R 9900 2200 60
 F3 "IN1" I L 9050 2200 60
@@
 U 5A019746
 F0 "Sheet5A019745" 60
-F1 "vn5e010ah.sch" 60
+F1 "vn5e010ah_double.sch" 60
 F2 "OUT1" O R 9900 2700 60
 F3 "IN1" I L 9050 2700 60
