File: hw/vn5e010ah_double.sch (KiCad schematic (older format))
At the start: 5 parts, among them U701 VN5E010AH, U702 VN5E010AH

Commit message: Drawing pcb 4.0.0
Parts:
- removed D701: DIODE_RS07J-GS18, usevolt:DO219AB, symbol usevolt:DIODE_RS07J-GS18
- added D5: ZENER_MM3Z3V6T1G, usevolt:SOD-323, symbol usevolt:ZENER_MM3Z3V6T1G
- added R3: 10K, yageo:0603, symbol yageo:10K
Connections:
- net GND: now also D5.2, R3.1 (R1)
- net OUT1: now also R3.2 (R2)
- net SENSE1: now also D5.1
Changed lines of the file:
@@
 Wire Wire Line
 	5450 3300 5450 3400
-Wire Wire Line
-	5450 4100 5450 3850
 Connection ~ 5450 3600
 $Comp
@@
 L power:GND #PWR0106
 U 1 1 5B1A40B3
-P 5650 3900
-F 0 "#PWR0106" H 5650 3650 50  0001 C CNN
-F 1 "GND" H 5655 3727 50  0000 C CNN
-F 2 "" H 5650 3900 50  0000 C CNN
-F 3 "" H 5650 3900 50  0000 C CNN
-	1    5650 3900
+P 5650 4550
+F 0 "#PWR0106" H 5650 4300 50  0001 C CNN
+F 1 "GND" H 5655 4377 50  0000 C CNN
+F 2 "" H 5650 4550 50  0000 C CNN
+F 3 "" H 5650 4550 50  0000 C CNN
+	1    5650 4550
 	1    0    0    -1
 $EndComp
@@
 Connection ~ 5650 3800
 Wire Wire Line
-	7100 3500 7600 3500
+	7100 3500 7350 3500
 Wire Wire Line
 	5450 3600 6300 3600
@@
 	4700 3850 4700 3900
 Wire Wire Line
-	5650 3800 5650 3900
+	5650 3800 5650 4450
 $Comp
 L usevolt:VN5E010AH U701
@@
 	1    0    0    -1
 $EndComp
-$Comp
-L usevolt:DIODE_RS07J-GS18 D701
-U 1 1 5B1C46E3
-P 5000 3850
-F 0 "D701" H 4950 3710 45  0000 C CNN
-F 1 "DIODE_RS07J-GS18" H 5020 3790 45  0001 L BNN
-F 2 "usevolt:DO219AB" H 5030 4000 20  0001 C CNN
-F 3 "http://www.vishay.com/docs/85742/rs07b.pdf" H 5020 3870 60  0001 C CNN
-F 4 "1864882" H 5620 4470 60  0001 C CNN "2nd Source Part Number"
-F 5 "Digi-Key" H 5320 4170 60  0001 C CNN "1st Source"
-F 6 "Farnell" H 5520 4370 60  0001 C CNN "2nd Source"
-F 7 "RS07J-GS18" H 5220 4070 60  0001 C CNN "Manufacturer Part Number"
-F 8 "RS07J-GS18-ND" H 5420 4270 60  0001 C CNN "1st Source Part Number"
-F 9 "Vishay Semiconductor Diodes Division" H 5120 3970 60  0001 C CNN "Manufacturer"
-	1    5000 3850
-	-1   0    0    1
-$EndComp
-Wire Wire Line
-	5200 3850 5450 3850
-Connection ~ 5450 3850
-Wire Wire Line
-	5450 3850 5450 3600
-$Comp
-L power:+3V3 #PWR0110
-U 1 1 5B1C4D66
-P 4850 3350
-F 0 "#PWR0110" H 4850 3200 50  0001 C CNN
-F 1 "+3V3" H 4865 3523 50  0000 C CNN
-F 2 "" H 4850 3350 50  0000 C CNN
-F 3 "" H 4850 3350 50  0000 C CNN
-	1    4850 3350
-	1    0    0    -1
-$EndComp
-Wire Wire Line
-	4850 3350 4850 3850
-Wire Wire Line
-	4850 3850 4900 3850
+Wire Wire Line
+	5450 3600 5450 4100
+$Comp
+L usevolt:ZENER_MM3Z3V6T1G D5
+U 1 1 5BAB3E6D
+P 5450 4250
+F 0 "D5" V 5375 4172 45  0000 R CNN
+F 1 "ZENER_MM3Z3V6T1G" H 5725 4625 45  0001 L BNN
+F 2 "usevolt:SOD-323" H 5425 4625 20  0001 C CNN
+F 3 "http://www.mouser.com/ds/2/308/MM3Z2V4T1-D-269162.pdf" H 5800 4825 60  0001 C CNN
+F 4 "Mouser" H 5770 4570 60  0001 C CNN "1st Source"
+F 5 "MM3Z3V6T1G" H 5670 4470 60  0001 C CNN "Manufacturer Part Number"
+F 6 "863-MM3Z3V6T1G" H 5870 4670 60  0001 C CNN "1st Source Part Number"
+F 7 "ON Semiconductor" H 5725 4725 60  0001 C CNN "Manufacturer"
+	1    5450 4250
+	0    -1   -1   0
+$EndComp
+Wire Wire Line
+	5450 4200 5450 4100
+Connection ~ 5450 4100
+Wire Wire Line
+	5450 4450 5650 4450
+Connection ~ 5650 4450
+Wire Wire Line
+	5650 4450 5650 4550
+$Comp
+L yageo:10K R3
+U 1 1 5BAB6B29
+P 7350 3750
+F 0 "R3" V 7358 3808 45  0000 L CNN
+F 1 "10K" V 7442 3808 45  0000 L CNN
+F 2 "yageo:0603" H 7380 3900 20  0001 C CNN
+F 3 "" H 7319 3789 60  0001 C CNN
+F 4 "" H 7719 4189 60  0001 C CNN "1st Source Part Number"
+F 5 "Digikey" H 7619 4089 60  0001 C CNN "1st Source"
+F 6 "RC0603FR-0710KL" H 7519 3989 60  0001 C CNN "Manufacturer Part Number"
+F 7 "YAGEO" H 7419 3889 60  0001 C CNN "Manufacturer"
+	1    7350 3750
+	0    1    1    0
+$EndComp
+Wire Wire Line
+	7350 3650 7350 3500
+Connection ~ 7350 3500
+Wire Wire Line
+	7350 3500 7600 3500
+$Comp
+L power:GND #PWR0109
+U 1 1 5BAB71FB
+P 7350 4050
+F 0 "#PWR0109" H 7350 3800 50  0001 C CNN
+F 1 "GND" H 7355 3877 50  0000 C CNN
+F 2 "" H 7350 4050 50  0000 C CNN
+F 3 "" H 7350 4050 50  0000 C CNN
+	1    7350 4050
+	1    0    0    -1
+$EndComp
+Wire Wire Line
+	7350 4050 7350 3950
 $EndSCHEMATC

Commit message: pcb 3.6.0 created, with double fets in work & drive lights
Parts:
- removed D5: ZENER_MM3Z3V6T1G, usevolt:SOD-323, symbol usevolt:ZENER_MM3Z3V6T1G
- removed R3: 10K, yageo:0603, symbol yageo:10K
- removed R702: 1K, yageo:0603, symbol yageo:1K
- added D8: ZENER_MM3Z3V6T1G, usevolt:SOD-323, symbol usevolt:ZENER_MM3Z3V6T1G
- added R1203: 1K, yageo:0603, symbol yageo:1K
- added R6: 10K, yageo:0603, symbol yageo:10K
- renumbered R701 to R1, U701 to U1201, U702 to U1202
Connections:
- net GND: now also D8.2, R1203.2 (R2), R6.1 (R1)
- net OUT1: now also R6.2 (R2)
- net SENSE1: now also D8.1, R1203.1 (R1)
