File: hw/vnd5050.sch (KiCad schematic (older format))
At the start: 5 parts, among them U401 VND5050AJTR-E

Commit message: hw 3.3 created
Changed lines of the file:
@@
 AR Path="/5A015FC0/59D8088A" Ref="U401"  Part="1"
 AR Path="/5A02A41F/59D8088A" Ref="U901"  Part="1"
-F 0 "U401" H 4700 4447 60  0000 C CNN
+F 0 "U901" H 4700 4447 60  0000 C CNN
 F 1 "VND5050AJTR-E" H 4700 4341 60  0000 C CNN
 F 2 "usevolt:PowerSSO-12" H 4600 4400 60  0001 C CNN
@@
 P 5250 3650
 AR Path="/5A015FC0/59D808C7" Ref="#PWR402"  Part="1"
-AR Path="/5A02A41F/59D808C7" Ref="#PWR902"  Part="1"
-F 0 "#PWR402" H 5250 3500 50  0001 C CNN
+AR Path="/5A02A41F/59D808C7" Ref="#PWR802"  Part="1"
+F 0 "#PWR802" H 5250 3500 50  0001 C CNN
 F 1 "VDD" H 5267 3823 50  0000 C CNN
 F 2 "" H 5250 3650 50  0000 C CNN
@@
 P 3600 4450
 AR Path="/5A015FC0/59D86DC2" Ref="#PWR401"  Part="1"
-AR Path="/5A02A41F/59D86DC2" Ref="#PWR901"  Part="1"
-F 0 "#PWR401" H 3600 4200 50  0001 C CNN
+AR Path="/5A02A41F/59D86DC2" Ref="#PWR801"  Part="1"
+F 0 "#PWR801" H 3600 4200 50  0001 C CNN
 F 1 "GND" H 3605 4277 50  0000 C CNN
 F 2 "" H 3600 4450 50  0000 C CNN
@@
 AR Path="/5A015FC0/59D88771" Ref="R402"  Part="1"
 AR Path="/5A02A41F/59D88771" Ref="R902"  Part="1"
-F 0 "R402" H 3850 4284 45  0000 C CNN
+F 0 "R902" H 3850 4284 45  0000 C CNN
 F 1 "390" H 3850 4200 45  0000 C CNN
 F 2 "yageo:0603" H 3830 4250 20  0001 C CNN
@@
 AR Path="/5A015FC0/59D88845" Ref="R401"  Part="1"
 AR Path="/5A02A41F/59D88845" Ref="R901"  Part="1"
-F 0 "R401" H 3850 4084 45  0000 C CNN
+F 0 "R901" H 3850 4084 45  0000 C CNN
 F 1 "390" H 3850 4000 45  0000 C CNN
 F 2 "yageo:0603" H 3830 4050 20  0001 C CNN
@@
 AR Path="/5A015FC0/5A05950C" Ref="R403"  Part="1"
 AR Path="/5A02A41F/5A05950C" Ref="R903"  Part="1"
-F 0 "R403" H 3450 4084 45  0000 C CNN
+F 0 "R903" H 3450 4084 45  0000 C CNN
 F 1 "1K" H 3450 4000 45  0000 C CNN
 F 2 "yageo:0603" H 3430 4050 20  0001 C CNN
@@
 AR Path="/5A015FC0/5A059568" Ref="R404"  Part="1"
 AR Path="/5A02A41F/5A059568" Ref="R904"  Part="1"
-F 0 "R404" H 3450 4284 45  0000 C CNN
+F 0 "R904" H 3450 4284 45  0000 C CNN
 F 1 "1K" H 3450 4200 45  0000 C CNN
 F 2 "yageo:0603" H 3430 4250 20  0001 C CNN

Commit message: making modifications to pcb...
Parts:
- removed R401, R402: 390, yageo:0603, symbol 390
- added D801, D802: DIODE_RS07J-GS18, usevolt:DO219AB, symbol usevolt:DIODE_RS07J-GS18
- added R801, R802: 1K, yageo:0603, symbol yageo:1K
- R403, R404: symbol 1K -> yageo:1K
- U401: symbol VND5050AJTR-E -> usevolt:VND5050AJTR-E
Connections:
- net GND: now also R801.2 (R2), R802.2 (R2)
- net SENSE1: now also D801.P$1 (P), R801.1 (R1)
- net SENSE2: now also D802.P$1 (P), R802.1 (R1)
- new net +3V3: D801.P$2 (N), D802.P$2 (N)
Changed lines of the file:
@@
-EESchema Schematic File Version 2
-LIBS:csb-rescue
-LIBS:kemet
-LIBS:power
-LIBS:usevolt
-LIBS:wurth_elektronik_LED
-LIBS:yageo
+EESchema Schematic File Version 4
 LIBS:csb-cache
 EELAYER 26 0
@@
 $Descr A4 11693 8268
 encoding utf-8
-Sheet 4 8
+Sheet 8 8
 Title ""
 Date ""
@@
 SENSE2
 $Comp
-L VND5050AJTR-E U401
+L usevolt:VND5050AJTR-E U401
 U 1 1 59D8088A
 P 4600 4000
 AR Path="/5A015FC0/59D8088A" Ref="U401"  Part="1"
 AR Path="/5A02A41F/59D8088A" Ref="U901"  Part="1"
-F 0 "U901" H 4700 4447 60  0000 C CNN
+F 0 "U401" H 4700 4447 60  0000 C CNN
 F 1 "VND5050AJTR-E" H 4700 4341 60  0000 C CNN
 F 2 "usevolt:PowerSSO-12" H 4600 4400 60  0001 C CNN
@@
 $EndComp
 $Comp
-L VDD #PWR402
+L power:VDD #PWR0402
 U 1 1 59D808C7
 P 5250 3650
-AR Path="/5A015FC0/59D808C7" Ref="#PWR402"  Part="1"
-AR Path="/5A02A41F/59D808C7" Ref="#PWR802"  Part="1"
-F 0 "#PWR802" H 5250 3500 50  0001 C CNN
+AR Path="/5A015FC0/59D808C7" Ref="#PWR0402"  Part="1"
+AR Path="/5A02A41F/59D808C7" Ref="#PWR0802"  Part="1"
+F 0 "#PWR0402" H 5250 3500 50  0001 C CNN
 F 1 "VDD" H 5267 3823 50  0000 C CNN
 F 2 "" H 5250 3650 50  0000 C CNN
@@
 $EndComp
 Wire Wire Line
-	5250 3650 5250 4000
+	5250 3650 5250 3800
 Wire Wire Line
 	5250 3800 5100 3800
@@
 Connection ~ 5250 3900
 Wire Wire Line
-	5100 4100 5800 4100
+	5100 4100 5250 4100
 Wire Wire Line
 	5100 4200 5250 4200
@@
 Connection ~ 5250 4100
 Wire Wire Line
-	5100 4400 5800 4400
+	5100 4400 5250 4400
 Wire Wire Line
 	5100 4300 5250 4300
@@
 Connection ~ 5250 4400
 Wire Wire Line
-	3200 3800 4300 3800
-Wire Wire Line
-	3200 4000 4300 4000
-$Comp
-L GND #PWR401
+	3200 3800 3300 3800
+Wire Wire Line
+	3200 4000 3300 4000
+$Comp
+L power:GND #PWR0401
 U 1 1 59D86DC2
 P 3600 4450
-AR Path="/5A015FC0/59D86DC2" Ref="#PWR401"  Part="1"
-AR Path="/5A02A41F/59D86DC2" Ref="#PWR801"  Part="1"
-F 0 "#PWR801" H 3600 4200 50  0001 C CNN
+AR Path="/5A015FC0/59D86DC2" Ref="#PWR0401"  Part="1"
+AR Path="/5A02A41F/59D86DC2" Ref="#PWR0801"  Part="1"
+F 0 "#PWR0401" H 3600 4200 50  0001 C CNN
 F 1 "GND" H 3605 4277 50  0000 C CNN
 F 2 "" H 3600 4450 50  0000 C CNN
@@
 $EndComp
 Wire Wire Line
-	3600 3900 3600 4450
+	3600 3900 3600 4100
 Wire Wire Line
 	3600 4300 4300 4300
-$Comp
-L 390 R402
-U 1 1 59D88771
-P 3800 4100
-AR Path="/5A015FC0/59D88771" Ref="R402"  Part="1"
-AR Path="/5A02A41F/59D88771" Ref="R902"  Part="1"
-F 0 "R902" H 3850 4284 45  0000 C CNN
-F 1 "390" H 3850 4200 45  0000 C CNN
-F 2 "yageo:0603" H 3830 4250 20  0001 C CNN
-F 3 "" H 3769 4139 60  0001 C CNN
-F 4 "" H 4169 4539 60  0001 C CNN "1st Source Part Number"
-F 5 "Digikey" H 4069 4439 60  0001 C CNN "1st Source"
-F 6 "RC0603FR-07390RL" H 3969 4339 60  0001 C CNN "Manufacturer Part Number"
-F 7 "YAGEO" H 3869 4239 60  0001 C CNN "Manufacturer"
-	1    3800 4100
-	1    0    0    -1
-$EndComp
-$Comp
-L 390 R401
-U 1 1 59D88845
-P 3800 3900
-AR Path="/5A015FC0/59D88845" Ref="R401"  Part="1"
-AR Path="/5A02A41F/59D88845" Ref="R901"  Part="1"
-F 0 "R901" H 3850 4084 45  0000 C CNN
-F 1 "390" H 3850 4000 45  0000 C CNN
-F 2 "yageo:0603" H 3830 4050 20  0001 C CNN
-F 3 "" H 3769 3939 60  0001 C CNN
-F 4 "" H 4169 4339 60  0001 C CNN "1st Source Part Number"
-F 5 "Digikey" H 4069 4239 60  0001 C CNN "1st Source"
-F 6 "RC0603FR-07390RL" H 3969 4139 60  0001 C CNN "Manufacturer Part Number"
-F 7 "YAGEO" H 3869 4039 60  0001 C CNN "Manufacturer"
-	1    3800 3900
-	1    0    0    -1
-$EndComp
 Wire Wire Line
 	3700 3900 3600 3900
@@
 Connection ~ 3600 4100
 Wire Wire Line
-	4000 4100 4300 4100
-Wire Wire Line
-	4000 3900 4300 3900
-Wire Wire Line
-	3200 4200 4150 4200
+	4000 4100 4150 4100
+Wire Wire Line
+	4000 3900 4150 3900
+Wire Wire Line
+	3200 4200 3750 4200
 Wire Wire Line
 	4150 4200 4150 4100
@@
 	4150 3900 4150 3700
 Wire Wire Line
-	4150 3700 3200 3700
+	4150 3700 3700 3700
 Connection ~ 4150 3900
 $Comp
-L 1K R403
+L yageo:1K R403
 U 1 1 5A05950C
 P 3400 3900
 AR Path="/5A015FC0/5A05950C" Ref="R403"  Part="1"
 AR Path="/5A02A41F/5A05950C" Ref="R903"  Part="1"
-F 0 "R903" H 3450 4084 45  0000 C CNN
+F 0 "R403" H 3450 4084 45  0000 C CNN
 F 1 "1K" H 3450 4000 45  0000 C CNN
 F 2 "yageo:0603" H 3430 4050 20  0001 C CNN
@@
 $EndComp
 $Comp
-L 1K R404
+L yageo:1K R404
 U 1 1 5A059568
 P 3400 4100
 AR Path="/5A015FC0/5A059568" Ref="R404"  Part="1"
 AR Path="/5A02A41F/5A059568" Ref="R904"  Part="1"
-F 0 "R904" H 3450 4284 45  0000 C CNN
+F 0 "R404" H 3450 4284 45  0000 C CNN
 F 1 "1K" H 3450 4200 45  0000 C CNN
 F 2 "yageo:0603" H 3430 4250 20  0001 C CNN
@@
 Connection ~ 3300 4000
 Connection ~ 3600 3900
+Wire Wire Line
+	5250 3800 5250 3900
+Wire Wire Line
+	5250 3900 5250 4000
+Wire Wire Line
+	5250 4100 5800 4100
+Wire Wire Line
+	5250 4400 5800 4400
+Wire Wire Line
+	3600 4300 3600 4450
+Wire Wire Line
+	3600 4100 3600 4300
+Wire Wire Line
+	4150 4100 4300 4100
+Wire Wire Line
+	4150 3900 4300 3900
+Wire Wire Line
+	3300 3800 4300 3800
+Wire Wire Line
+	3300 4000 4300 4000
+$Comp
+L yageo:1K R801
+U 1 1 5B1C6487
+P 3800 3900
+AR Path="/5A02A41F/5B1C6487" Ref="R801"  Part="1"
+AR Path="/5A015FC0/5B1C6487" Ref="R401"  Part="1"
+F 0 "R401" H 3850 4084 45  0000 C CNN
+F 1 "1K" H 3850 4000 45  0000 C CNN
+F 2 "yageo:0603" H 3830 4050 20  0001 C CNN
+F 3 "" H 3769 3939 60  0001 C CNN
+F 4 "" H 4169 4339 60  0001 C CNN "1st Source Part Number"
+F 5 "Digikey" H 4069 4239 60  0001 C CNN "1st Source"
+F 6 "RC0603FR-071KL" H 3969 4139 60  0001 C CNN "Manufacturer Part Number"
+F 7 "YAGEO" H 3869 4039 60  0001 C CNN "Manufacturer"
+	1    3800 3900
+	1    0    0    -1
+$EndComp
+$Comp
+L yageo:1K R802
+U 1 1 5B1C64C1
+P 3800 4100
+AR Path="/5A02A41F/5B1C64C1" Ref="R802"  Part="1"
+AR Path="/5A015FC0/5B1C64C1" Ref="R402"  Part="1"
+F 0 "R402" H 3850 4284 45  0000 C CNN
+F 1 "1K" H 3850 4200 45  0000 C CNN
+F 2 "yageo:0603" H 3830 4250 20  0001 C CNN
+F 3 "" H 3769 4139 60  0001 C CNN
+F 4 "" H 4169 4539 60  0001 C CNN "1st Source Part Number"
+F 5 "Digikey" H 4069 4439 60  0001 C CNN "1st Source"
+F 6 "RC0603FR-071KL" H 3969 4339 60  0001 C CNN "Manufacturer Part Number"
+F 7 "YAGEO" H 3869 4239 60  0001 C CNN "Manufacturer"
+	1    3800 4100
+	1    0    0    -1
+$EndComp
+$Comp
+L usevolt:DIODE_RS07J-GS18 D801
+U 1 1 5B1C66B1
+P 3900 3500
+AR Path="/5A02A41F/5B1C66B1" Ref="D801"  Part="1"
+AR Path="/5A015FC0/5B1C66B1" Ref="D401"  Part="1"
+F 0 "D401" H 3850 3360 45  0000 C CNN
+F 1 "DIODE_RS07J-GS18" H 3920 3440 45  0001 L BNN
+F 2 "usevolt:DO219AB" H 3930 3650 20  0001 C CNN
+F 3 "http://www.vishay.com/docs/85742/rs07b.pdf" H 3920 3520 60  0001 C CNN
+F 4 "1864882" H 4520 4120 60  0001 C CNN "2nd Source Part Number"
+F 5 "Digi-Key" H 4220 3820 60  0001 C CNN "1st Source"
+F 6 "Farnell" H 4420 4020 60  0001 C CNN "2nd Source"
+F 7 "RS07J-GS18" H 4120 3720 60  0001 C CNN "Manufacturer Part Number"
+F 8 "RS07J-GS18-ND" H 4320 3920 60  0001 C CNN "1st Source Part Number"
+F 9 "Vishay Semiconductor Diodes Division" H 4020 3620 60  0001 C CNN "Manufacturer"
+	1    3900 3500
+	1    0    0    -1
+$EndComp
+$Comp
+L usevolt:DIODE_RS07J-GS18 D802
+U 1 1 5B1CE776
+P 3950 4450
+AR Path="/5A02A41F/5B1CE776" Ref="D802"  Part="1"
+AR Path="/5A015FC0/5B1CE776" Ref="D402"  Part="1"
+F 0 "D402" H 3900 4310 45  0000 C CNN
+F 1 "DIODE_RS07J-GS18" H 3970 4390 45  0001 L BNN
+F 2 "usevolt:DO219AB" H 3980 4600 20  0001 C CNN
+F 3 "http://www.vishay.com/docs/85742/rs07b.pdf" H 3970 4470 60  0001 C CNN
+F 4 "1864882" H 4570 5070 60  0001 C CNN "2nd Source Part Number"
+F 5 "Digi-Key" H 4270 4770 60  0001 C CNN "1st Source"
+F 6 "Farnell" H 4470 4970 60  0001 C CNN "2nd Source"
+F 7 "RS07J-GS18" H 4170 4670 60  0001 C CNN "Manufacturer Part Number"
+F 8 "RS07J-GS18-ND" H 4370 4870 60  0001 C CNN "1st Source Part Number"
+F 9 "Vishay Semiconductor Diodes Division" H 4070 4570 60  0001 C CNN "Manufacturer"
+	1    3950 4450
+	1    0    0    -1
+$EndComp
+Wire Wire Line
+	4050 4450 4100 4450
+Wire Wire Line
+	4100 4450 4100 3500
+Wire Wire Line
+	4100 3500 4000 3500
+Wire Wire Line
+	3750 4450 3750 4200
+Connection ~ 3750 4200
+Wire Wire Line
+	3750 4200 4150 4200
+Wire Wire Line
+	3700 3500 3700 3700
+Connection ~ 3700 3700
+Wire Wire Line
+	3700 3700 3200 3700
+$Comp
+L power:+3V3 #PWR0111
+U 1 1 5B1D1455
+P 4100 3500
+AR Path="/5A02A41F/5B1D1455" Ref="#PWR0111"  Part="1"
+AR Path="/5A015FC0/5B1D1455" Ref="#PWR0107"  Part="1"
+F 0 "#PWR0107" H 4100 3350 50  0001 C CNN
+F 1 "+3V3" H 4115 3673 50  0000 C CNN
+F 2 "" H 4100 3500 50  0000 C CNN
+F 3 "" H 4100 3500 50  0000 C CNN
+	1    4100 3500
+	1    0    0    -1
+$EndComp
+Connection ~ 4100 3500
 $EndSCHEMATC

Commit message: Drawing pcb 4.0.0
Parts:
- removed D801, D802: DIODE_RS07J-GS18, usevolt:DO219AB, symbol usevolt:DIODE_RS07J-GS18
- added D6, D7: ZENER_MM3Z3V6T1G, usevolt:SOD-323, symbol usevolt:ZENER_MM3Z3V6T1G
Connections:
- net GND: now also D6.2, D7.2
- net SENSE1: now also D6.1
- net SENSE2: now also D7.1
Other:
- moved on the sheet: R801, R802
Changed lines of the file:
@@
 AR Path="/5A015FC0/59D8088A" Ref="U401"  Part="1"
 AR Path="/5A02A41F/59D8088A" Ref="U901"  Part="1"
-F 0 "U401" H 4700 4447 60  0000 C CNN
+F 0 "U901" H 4700 4447 60  0000 C CNN
 F 1 "VND5050AJTR-E" H 4700 4341 60  0000 C CNN
 F 2 "usevolt:PowerSSO-12" H 4600 4400 60  0001 C CNN
@@
 AR Path="/5A015FC0/59D808C7" Ref="#PWR0402"  Part="1"
 AR Path="/5A02A41F/59D808C7" Ref="#PWR0802"  Part="1"
-F 0 "#PWR0402" H 5250 3500 50  0001 C CNN
+F 0 "#PWR0802" H 5250 3500 50  0001 C CNN
 F 1 "VDD" H 5267 3823 50  0000 C CNN
 F 2 "" H 5250 3650 50  0000 C CNN
@@
 L power:GND #PWR0401
 U 1 1 59D86DC2
-P 3600 4450
+P 3600 4900
 AR Path="/5A015FC0/59D86DC2" Ref="#PWR0401"  Part="1"
 AR Path="/5A02A41F/59D86DC2" Ref="#PWR0801"  Part="1"
-F 0 "#PWR0401" H 3600 4200 50  0001 C CNN
-F 1 "GND" H 3605 4277 50  0000 C CNN
-F 2 "" H 3600 4450 50  0000 C CNN
-F 3 "" H 3600 4450 50  0000 C CNN
-	1    3600 4450
-	1    0    0    -1
-$EndComp
-Wire Wire Line
-	3600 3900 3600 4100
+F 0 "#PWR0801" H 3600 4650 50  0001 C CNN
+F 1 "GND" H 3605 4727 50  0000 C CNN
+F 2 "" H 3600 4900 50  0000 C CNN
+F 3 "" H 3600 4900 50  0000 C CNN
+	1    3600 4900
+	1    0    0    -1
+$EndComp
 Wire Wire Line
 	3600 4300 4300 4300
 Wire Wire Line
-	3700 3900 3600 3900
-Connection ~ 3600 4300
-Wire Wire Line
-	3700 4100 3600 4100
-Connection ~ 3600 4100
-Wire Wire Line
-	4000 4100 4150 4100
-Wire Wire Line
-	4000 3900 4150 3900
-Wire Wire Line
-	3200 4200 3750 4200
-Wire Wire Line
 	4150 4200 4150 4100
-Connection ~ 4150 4100
 Wire Wire Line
 	4150 3900 4150 3700
-Wire Wire Line
-	4150 3700 3700 3700
-Connection ~ 4150 3900
 $Comp
 L yageo:1K R403
@@
 AR Path="/5A015FC0/5A05950C" Ref="R403"  Part="1"
 AR Path="/5A02A41F/5A05950C" Ref="R903"  Part="1"
-F 0 "R403" H 3450 4084 45  0000 C CNN
+F 0 "R903" H 3450 4084 45  0000 C CNN
 F 1 "1K" H 3450 4000 45  0000 C CNN
 F 2 "yageo:0603" H 3430 4050 20  0001 C CNN
@@
 AR Path="/5A015FC0/5A059568" Ref="R404"  Part="1"
 AR Path="/5A02A41F/5A059568" Ref="R904"  Part="1"
-F 0 "R404" H 3450 4284 45  0000 C CNN
+F 0 "R904" H 3450 4284 45  0000 C CNN
 F 1 "1K" H 3450 4200 45  0000 C CNN
 F 2 "yageo:0603" H 3430 4250 20  0001 C CNN
@@
 	3300 4000 3300 4100
 Connection ~ 3300 4000
-Connection ~ 3600 3900
 Wire Wire Line
 	5250 3800 5250 3900
@@
 	5250 4400 5800 4400
 Wire Wire Line
-	3600 4300 3600 4450
-Wire Wire Line
-	3600 4100 3600 4300
+	3600 4300 3600 4850
 Wire Wire Line
 	4150 4100 4300 4100
@@
 L yageo:1K R801
 U 1 1 5B1C6487
-P 3800 3900
+P 3850 3900
 AR Path="/5A02A41F/5B1C6487" Ref="R801"  Part="1"
 AR Path="/5A015FC0/5B1C6487" Ref="R401"  Part="1"
-F 0 "R401" H 3850 4084 45  0000 C CNN
-F 1 "1K" H 3850 4000 45  0000 C CNN
-F 2 "yageo:0603" H 3830 4050 20  0001 C CNN
-F 3 "" H 3769 3939 60  0001 C CNN
-F 4 "" H 4169 4339 60  0001 C CNN "1st Source Part Number"
-F 5 "Digikey" H 4069 4239 60  0001 C CNN "1st Source"
-F 6 "RC0603FR-071KL" H 3969 4139 60  0001 C CNN "Manufacturer Part Number"
-F 7 "YAGEO" H 3869 4039 60  0001 C CNN "Manufacturer"
-	1    3800 3900
+F 0 "R801" H 3900 4084 45  0000 C CNN
+F 1 "1K" H 3900 4000 45  0000 C CNN
+F 2 "yageo:0603" H 3880 4050 20  0001 C CNN
+F 3 "" H 3819 3939 60  0001 C CNN
+F 4 "" H 4219 4339 60  0001 C CNN "1st Source Part Number"
+F 5 "Digikey" H 4119 4239 60  0001 C CNN "1st Source"
+F 6 "RC0603FR-071KL" H 4019 4139 60  0001 C CNN "Manufacturer Part Number"
+F 7 "YAGEO" H 3919 4039 60  0001 C CNN "Manufacturer"
+	1    3850 3900
 	1    0    0    -1
 $EndComp
@@
 L yageo:1K R802
 U 1 1 5B1C64C1
-P 3800 4100
+P 3850 4100
 AR Path="/5A02A41F/5B1C64C1" Ref="R802"  Part="1"
 AR Path="/5A015FC0/5B1C64C1" Ref="R402"  Part="1"
-F 0 "R402" H 3850 4284 45  0000 C CNN
-F 1 "1K" H 3850 4200 45  0000 C CNN
-F 2 "yageo:0603" H 3830 4250 20  0001 C CNN
-F 3 "" H 3769 4139 60  0001 C CNN
-F 4 "" H 4169 4539 60  0001 C CNN "1st Source Part Number"
-F 5 "Digikey" H 4069 4439 60  0001 C CNN "1st Source"
-F 6 "RC0603FR-071KL" H 3969 4339 60  0001 C CNN "Manufacturer Part Number"
-F 7 "YAGEO" H 3869 4239 60  0001 C CNN "Manufacturer"
-	1    3800 4100
-	1    0    0    -1
-$EndComp
-$Comp
-L usevolt:DIODE_RS07J-GS18 D801
-U 1 1 5B1C66B1
-P 3900 3500
-AR Path="/5A02A41F/5B1C66B1" Ref="D801"  Part="1"
-AR Path="/5A015FC0/5B1C66B1" Ref="D401"  Part="1"
-F 0 "D401" H 3850 3360 45  0000 C CNN
-F 1 "DIODE_RS07J-GS18" H 3920 3440 45  0001 L BNN
-F 2 "usevolt:DO219AB" H 3930 3650 20  0001 C CNN
-F 3 "http://www.vishay.com/docs/85742/rs07b.pdf" H 3920 3520 60  0001 C CNN
-F 4 "1864882" H 4520 4120 60  0001 C CNN "2nd Source Part Number"
-F 5 "Digi-Key" H 4220 3820 60  0001 C CNN "1st Source"
-F 6 "Farnell" H 4420 4020 60  0001 C CNN "2nd Source"
-F 7 "RS07J-GS18" H 4120 3720 60  0001 C CNN "Manufacturer Part Number"
-F 8 "RS07J-GS18-ND" H 4320 3920 60  0001 C CNN "1st Source Part Number"
-F 9 "Vishay Semiconductor Diodes Division" H 4020 3620 60  0001 C CNN "Manufacturer"
-	1    3900 3500
-	1    0    0    -1
-$EndComp
-$Comp
-L usevolt:DIODE_RS07J-GS18 D802
-U 1 1 5B1CE776
-P 3950 4450
-AR Path="/5A02A41F/5B1CE776" Ref="D802"  Part="1"
-AR Path="/5A015FC0/5B1CE776" Ref="D402"  Part="1"
-F 0 "D402" H 3900 4310 45  0000 C CNN
-F 1 "DIODE_RS07J-GS18" H 3970 4390 45  0001 L BNN
-F 2 "usevolt:DO219AB" H 3980 4600 20  0001 C CNN
-F 3 "http://www.vishay.com/docs/85742/rs07b.pdf" H 3970 4470 60  0001 C CNN
-F 4 "1864882" H 4570 5070 60  0001 C CNN "2nd Source Part Number"
-F 5 "Digi-Key" H 4270 4770 60  0001 C CNN "1st Source"
-F 6 "Farnell" H 4470 4970 60  0001 C CNN "2nd Source"
-F 7 "RS07J-GS18" H 4170 4670 60  0001 C CNN "Manufacturer Part Number"
-F 8 "RS07J-GS18-ND" H 4370 4870 60  0001 C CNN "1st Source Part Number"
-F 9 "Vishay Semiconductor Diodes Division" H 4070 4570 60  0001 C CNN "Manufacturer"
-	1    3950 4450
-	1    0    0    -1
-$EndComp
-Wire Wire Line
-	4050 4450 4100 4450
-Wire Wire Line
-	4100 4450 4100 3500
-Wire Wire Line
-	4100 3500 4000 3500
-Wire Wire Line
-	3750 4450 3750 4200
-Connection ~ 3750 4200
-Wire Wire Line
-	3750 4200 4150 4200
-Wire Wire Line
-	3700 3500 3700 3700
+F 0 "R802" H 3900 4284 45  0000 C CNN
+F 1 "1K" H 3900 4200 45  0000 C CNN
+F 2 "yageo:0603" H 3880 4250 20  0001 C CNN
+F 3 "" H 3819 4139 60  0001 C CNN
+F 4 "" H 4219 4539 60  0001 C CNN "1st Source Part Number"
+F 5 "Digikey" H 4119 4439 60  0001 C CNN "1st Source"
+F 6 "RC0603FR-071KL" H 4019 4339 60  0001 C CNN "Manufacturer Part Number"
+F 7 "YAGEO" H 3919 4239 60  0001 C CNN "Manufacturer"
+	1    3850 4100
+	1    0    0    -1
+$EndComp
+Wire Wire Line
+	3700 3700 3200 3700
+Wire Wire Line
+	4150 3700 3700 3700
 Connection ~ 3700 3700
-Wire Wire Line
-	3700 3700 3200 3700
-$Comp
-L power:+3V3 #PWR0111
-U 1 1 5B1D1455
-P 4100 3500
-AR Path="/5A02A41F/5B1D1455" Ref="#PWR0111"  Part="1"
-AR Path="/5A015FC0/5B1D1455" Ref="#PWR0107"  Part="1"
-F 0 "#PWR0107" H 4100 3350 50  0001 C CNN
-F 1 "+3V3" H 4115 3673 50  0000 C CNN
-F 2 "" H 4100 3500 50  0000 C CNN
-F 3 "" H 4100 3500 50  0000 C CNN
-	1    4100 3500
-	1    0    0    -1
-$EndComp
-Connection ~ 4100 3500
+$Comp
+L usevolt:ZENER_MM3Z3V6T1G D6
+U 1 1 5BAB973C
+P 3700 4550
+AR Path="/5A02A41F/5BAB973C" Ref="D6"  Part="1"
+AR Path="/5A015FC0/5BAB973C" Ref="D1"  Part="1"
+F 0 "D6" V 3625 4472 45  0000 R CNN
+F 1 "ZENER_MM3Z3V6T1G" H 3975 4925 45  0001 L BNN
+F 2 "usevolt:SOD-323" H 3675 4925 20  0001 C CNN
+F 3 "http://www.mouser.com/ds/2/308/MM3Z2V4T1-D-269162.pdf" H 4050 5125 60  0001 C CNN
+F 4 "Mouser" H 4020 4870 60  0001 C CNN "1st Source"
+F 5 "MM3Z3V6T1G" H 3920 4770 60  0001 C CNN "Manufacturer Part Number"
+F 6 "863-MM3Z3V6T1G" H 4120 4970 60  0001 C CNN "1st Source Part Number"
+F 7 "ON Semiconductor" H 3975 5025 60  0001 C CNN "Manufacturer"
+	1    3700 4550
+	0    -1   -1   0
+$EndComp
+Wire Wire Line
+	3200 4200 3950 4200
+$Comp
+L usevolt:ZENER_MM3Z3V6T1G D7
+U 1 1 5BAB9E63
+P 3950 4550
+AR Path="/5A02A41F/5BAB9E63" Ref="D7"  Part="1"
+AR Path="/5A015FC0/5BAB9E63" Ref="D2"  Part="1"
+F 0 "D7" V 3875 4472 45  0000 R CNN
+F 1 "ZENER_MM3Z3V6T1G" H 4225 4925 45  0001 L BNN
+F 2 "usevolt:SOD-323" H 3925 4925 20  0001 C CNN
+F 3 "http://www.mouser.com/ds/2/308/MM3Z2V4T1-D-269162.pdf" H 4300 5125 60  0001 C CNN
+F 4 "Mouser" H 4270 4870 60  0001 C CNN "1st Source"
+F 5 "MM3Z3V6T1G" H 4170 4770 60  0001 C CNN "Manufacturer Part Number"
+F 6 "863-MM3Z3V6T1G" H 4370 4970 60  0001 C CNN "1st Source Part Number"
+F 7 "ON Semiconductor" H 4225 5025 60  0001 C CNN "Manufacturer"
+	1    3950 4550
+	0    -1   -1   0
+$EndComp
+Wire Wire Line
+	3950 4500 3950 4200
+Connection ~ 3950 4200
+Wire Wire Line
+	3950 4200 4150 4200
+Wire Wire Line
+	3700 4750 3700 4850
+Wire Wire Line
+	3700 4850 3600 4850
+Connection ~ 3600 4850
+Wire Wire Line
+	3600 4850 3600 4900
+Wire Wire Line
+	3700 4850 3950 4850
+Wire Wire Line
+	3950 4850 3950 4750
+Connection ~ 3700 4850
+Wire Wire Line
+	3700 3700 3700 4500
+Wire Wire Line
+	4050 4100 4150 4100
+Connection ~ 4150 4100
+Wire Wire Line
+	4150 3900 4050 3900
+Connection ~ 4150 3900
+Wire Wire Line
+	3600 3900 3600 4100
+Wire Wire Line
+	3600 4100 3600 4300
+Connection ~ 3600 4100
+Connection ~ 3600 4300
+Wire Wire Line
+	3750 4100 3600 4100
+Wire Wire Line
+	3600 3900 3750 3900
+Connection ~ 3600 3900
 $EndSCHEMATC
